Commit message: add more integration with the web app

File: ros2_simulation/my_ws/src/articubot_one/description/camera.xacro (robot description, xacro)
@@ -4,5 +4,5 @@
         <parent link="chassis"/>
         <child link="camera_link"/>
-        <origin xyz="0.276 0 0.181" rpy="0 0.18 0"/>
+        <origin xyz="0.335 0 0.08" rpy="0 0 0"/>
     </joint>
     <link name="camera_link">
@@ -11,12 +11,5 @@
                 <box size="0.010 0.03 0.03"/>
             </geometry>
-            <material name="black"/>
-        </visual>
-        <visual>
-            <origin xyz="0 0 -0.05"/>
-            <geometry>
-                <cylinder radius="0.002" length="0.1"/>
-            </geometry>
-            <material name="black"/>
+            <material name="red"/>
         </visual>
     </link>
@@ -32,5 +25,5 @@
             <pose> 0 0 0 0 0 0 </pose>
             <visualize>true</visualize>
-            <update_rate>10</update_rate>
+            <update_rate>20</update_rate>
             <camera>
                 <horizontal_fov>1.089</horizontal_fov>

File: ros2_simulation/my_ws/src/articubot_one/description/distance_sensor.xacro (robot description, xacro)
@@ -4,5 +4,5 @@
         <parent link="chassis"/>
         <child link="distance_sensor_link"/>
-        <origin xyz="0.335 0 0.08" rpy="0 0 0"/>
+        <origin xyz="0.335 0.05 0.08" rpy="0 0 0"/>
     </joint>
     <link name="distance_sensor_link">
